File: pcb/crossfire_mk1.kicad_sch (KiCad schematic)
At the start: 44 parts, among them J1 USB_C_Receptacle_USB2.0, J6 Conn_01x05, J7 Conn_01x07, SW1 SW_Push_Dual, U1 W25Q16JVUXIQ_TR, U2 RP2040, U3 AP22953CW12-7, U4 RT6154AGQW, X1 ABM8-272-T3

Commit message: integrate debug and oled connectors
Parts:
- added J8: OLED_PWR_JMP, Connector_PinHeader_2.54mm:PinHeader_1x03_P2.54mm_Vertical, symbol Connector:Conn_01x03_Pin
- J6: value Conn_01x05 -> DEBUG_CONN
- J7: value Conn_01x07 -> OLED_CONN
- SW1: value SW_Push_Dual -> SW_RESET; footprint Button_Switch_THT:SW_PUSH_6mm -> project-fooprints:Sumida_CPFC6D36NP-100M06
Connections:
- net +3.3V: now also J8.3 (Pin_3)
- net +5V: now also J8.1 (Pin_1); no longer J7.2 (Pin_2)
- net led_status: now also U2.35 (GPIO23); no longer U2.37 (GPIO25)
- net oled_clk: now also U2.40 (GPIO28_ADC2)
- net oled_cs: now also U2.36 (GPIO24)
- net oled_data: now also U2.39 (GPIO27_ADC1)
- net oled_dc: now also U2.37 (GPIO25)
- net oled_reset: now also U2.38 (GPIO26_ADC0)
- net swd_clk: now also J6.2 (Pin_2); no longer J6.1 (Pin_1)
- net swd_io: now also J6.1 (Pin_1); no longer J6.2 (Pin_2)
- net usb4_vben: now also U2.29 (GPIO18); no longer U2.27 (GPIO16)
- net usbc1_vbus_pres: no longer U2.36 (GPIO24)
- new net oled_pwr: J7.2 (Pin_2), J8.2 (Pin_2)
